Commit message: Updated URDF, more launch params, yeeted uneeded

File: src/ah_urdf/urdf/left_thumb_only.urdf (robot description, URDF)
Before this commit: robot ability_hand, 4 links, 3 joints
Joints:
- joint thumb_q1: limit lower=-1.74 upper=0 effort=1.2 velocity=40.338888721 -> lower=-1.7453292519943295 upper=0 effort=1.2 velocity=40.338888721
- joint thumb_q2: limit lower=0 upper=1.74 effort=6.0 velocity=8.0677777442 -> lower=0 upper=1.7453292519943295 effort=6.0 velocity=8.0677777442

File: src/ah_urdf/urdf/right_thumb_only.urdf (robot description, URDF)
Before this commit: robot ability_hand, 4 links, 3 joints
Joints:
- joint thumb_q1: limit lower=-1.74 upper=0 effort=1.2 velocity=40.338888721 -> lower=-1.7453292519943295 upper=0 effort=1.2 velocity=40.338888721
- joint thumb_q2: limit lower=0 upper=1.74 effort=6.0 velocity=8.0677777442 -> lower=0 upper=1.7453292519943295 effort=6.0 velocity=8.0677777442
