Commit message: better offsets

File: src/ah_urdf/urdf/ability_hand_left_large.urdf (robot description, URDF)
Before this commit: robot ability_hand, 47 links, 46 joints
Joints:
- joint index_q2: limit lower=0.766 upper=2.61 effort=6.0 velocity=8.0677777442 -> lower=0.00 upper=1.844 effort=6.0 velocity=8.0677777442; mimic joint=index_q1 multiplier=1.05851325 offset=0.72349796 -> joint=index_q1 multiplier=1.05851325; origin xyz=38.472723e-3 3.257695e-3 0.000000e-3 rpy=0 0 0.084474 -> xyz=38.472723e-3 3.257695e-3 0.000000e-3 rpy=0 0 0.766
- joint middle_q2: limit lower=0.766 upper=2.61 effort=6.0 velocity=8.0677777442 -> lower=0.00 upper=1.844 effort=6.0 velocity=8.0677777442; mimic joint=middle_q1 multiplier=1.05851325 offset=0.72349796 -> joint=middle_q1 multiplier=1.05851325; origin xyz=38.472723e-3 3.257695e-3 0.000000 rpy=0 0 0.084474 -> xyz=38.472723e-3 3.257695e-3 0.000000 rpy=0 0 0.766
- joint pinky_q2: limit lower=0.766 upper=2.61 effort=6.0 velocity=8.0677777442 -> lower=0.00 upper=1.844 effort=6.0 velocity=8.0677777442; mimic joint=pinky_q1 multiplier=1.05851325 offset=0.72349796 -> joint=pinky_q1 multiplier=1.05851325; origin xyz=38.472723e-3 3.257695e-3 0.000000 rpy=0 0 0.084474 -> xyz=38.472723e-3 3.257695e-3 0.000000 rpy=0 0 0.766
- joint ring_q2: limit lower=0.766 upper=2.61 effort=6.0 velocity=8.0677777442 -> lower=0.00 upper=1.844 effort=6.0 velocity=8.0677777442; mimic joint=ring_q1 multiplier=1.05851325 offset=0.72349796 -> joint=ring_q1 multiplier=1.05851325; origin xyz=38.472723e-3 3.257695e-3 0.000000 rpy=0 0 0.084474 -> xyz=38.472723e-3 3.257695e-3 0.000000 rpy=0 0 0.766

File: src/ah_urdf/urdf/ability_hand_left_small.urdf (robot description, URDF)
Before this commit: robot ability_hand, 47 links, 46 joints
Joints:
- joint index_q2: limit lower=0.766 upper=2.61 effort=6.0 velocity=8.0677777442 -> lower=0.00 upper=1.844 effort=6.0 velocity=8.0677777442; mimic joint=index_q1 multiplier=1.05851325 offset=0.72349796 -> joint=index_q1 multiplier=1.05851325; origin xyz=38.472723e-3 3.257695e-3 0.000000e-3 rpy=0 0 0.084474 -> xyz=38.472723e-3 3.257695e-3 0.000000e-3 rpy=0 0 0.766
- joint middle_q2: limit lower=0.766 upper=2.61 effort=6.0 velocity=8.0677777442 -> lower=0.00 upper=1.844 effort=6.0 velocity=8.0677777442; mimic joint=middle_q1 multiplier=1.05851325 offset=0.72349796 -> joint=middle_q1 multiplier=1.05851325; origin xyz=38.472723e-3 3.257695e-3 0.000000 rpy=0 0 0.084474 -> xyz=38.472723e-3 3.257695e-3 0.000000 rpy=0 0 0.766
- joint pinky_q2: limit lower=0.766 upper=2.61 effort=6.0 velocity=8.0677777442 -> lower=0.00 upper=1.844 effort=6.0 velocity=8.0677777442; mimic joint=pinky_q1 multiplier=1.05851325 offset=0.72349796 -> joint=pinky_q1 multiplier=1.05851325; origin xyz=38.472723e-3 3.257695e-3 0.000000 rpy=0 0 0.084474 -> xyz=38.472723e-3 3.257695e-3 0.000000 rpy=0 0 0.766
- joint ring_q2: limit lower=0.766 upper=2.61 effort=6.0 velocity=8.0677777442 -> lower=0.00 upper=1.844 effort=6.0 velocity=8.0677777442; mimic joint=ring_q1 multiplier=1.05851325 offset=0.72349796 -> joint=ring_q1 multiplier=1.05851325; origin xyz=38.472723e-3 3.257695e-3 0.000000 rpy=0 0 0.084474 -> xyz=38.472723e-3 3.257695e-3 0.000000 rpy=0 0 0.766

File: src/ah_urdf/urdf/ability_hand_right_large.urdf (robot description, URDF)
Before this commit: robot ability_hand, 47 links, 46 joints
Joints:
- joint index_q2: limit lower=0.766 upper=2.61 effort=6.0 velocity=8.0677777442 -> lower=0.00 upper=1.844 effort=6.0 velocity=8.0677777442; mimic joint=index_q1 multiplier=1.05851325 offset=0.72349796 -> joint=index_q1 multiplier=1.05851325; origin xyz=38.472723e-3 3.257695e-3 0.000000e-3 rpy=0 0 0.084474 -> xyz=38.472723e-3 3.257695e-3 0.000000e-3 rpy=0 0 0.766
- joint middle_q2: limit lower=0.766 upper=2.61 effort=6.0 velocity=8.0677777442 -> lower=0.00 upper=1.844 effort=6.0 velocity=8.0677777442; mimic joint=middle_q1 multiplier=1.05851325 offset=0.72349796 -> joint=middle_q1 multiplier=1.05851325; origin xyz=38.472723e-3 3.257695e-3 0.000000 rpy=0 0 0.084474 -> xyz=38.472723e-3 3.257695e-3 0.000000 rpy=0 0 0.766
- joint pinky_q2: limit lower=0.766 upper=2.61 effort=6.0 velocity=8.0677777442 -> lower=0.00 upper=1.844 effort=6.0 velocity=8.0677777442; mimic joint=pinky_q1 multiplier=1.05851325 offset=0.72349796 -> joint=pinky_q1 multiplier=1.05851325; origin xyz=38.472723e-3 3.257695e-3 0.000000 rpy=0 0 0.084474 -> xyz=38.472723e-3 3.257695e-3 0.000000 rpy=0 0 0.766
- joint ring_q2: limit lower=0.766 upper=2.61 effort=6.0 velocity=8.0677777442 -> lower=0.00 upper=1.844 effort=6.0 velocity=8.0677777442; mimic joint=ring_q1 multiplier=1.05851325 offset=0.72349796 -> joint=ring_q1 multiplier=1.05851325; origin xyz=38.472723e-3 3.257695e-3 0.000000 rpy=0 0 0.084474 -> xyz=38.472723e-3 3.257695e-3 0.000000 rpy=0 0 0.766

File: src/ah_urdf/urdf/ability_hand_right_large_no_fsr.urdf (robot description, URDF)
Before this commit: robot ability_hand, 17 links, 16 joints
Joints:
- joint index_q2: limit lower=0.766 upper=2.61 effort=6.0 velocity=8.0677777442 -> lower=0.00 upper=1.844 effort=6.0 velocity=8.0677777442; mimic joint=index_q1 multiplier=1.05851325 offset=0.72349796 -> joint=index_q1 multiplier=1.05851325; origin xyz=38.472723e-3 3.257695e-3 0.000000e-3 rpy=0 0 0.084474 -> xyz=38.472723e-3 3.257695e-3 0.000000e-3 rpy=0 0 0.766
- joint middle_q2: limit lower=0.766 upper=2.61 effort=6.0 velocity=8.0677777442 -> lower=0.00 upper=1.844 effort=6.0 velocity=8.0677777442; mimic joint=middle_q1 multiplier=1.05851325 offset=0.72349796 -> joint=middle_q1 multiplier=1.05851325; origin xyz=38.472723e-3 3.257695e-3 0.000000 rpy=0 0 0.084474 -> xyz=38.472723e-3 3.257695e-3 0.000000 rpy=0 0 0.766
- joint pinky_q2: limit lower=0.766 upper=2.61 effort=6.0 velocity=8.0677777442 -> lower=0.00 upper=1.844 effort=6.0 velocity=8.0677777442; mimic joint=pinky_q1 multiplier=1.05851325 offset=0.72349796 -> joint=pinky_q1 multiplier=1.05851325; origin xyz=38.472723e-3 3.257695e-3 0.000000 rpy=0 0 0.084474 -> xyz=38.472723e-3 3.257695e-3 0.000000 rpy=0 0 0.766
- joint ring_q2: limit lower=0.766 upper=2.61 effort=6.0 velocity=8.0677777442 -> lower=0.00 upper=1.844 effort=6.0 velocity=8.0677777442; mimic joint=ring_q1 multiplier=1.05851325 offset=0.72349796 -> joint=ring_q1 multiplier=1.05851325; origin xyz=38.472723e-3 3.257695e-3 0.000000 rpy=0 0 0.084474 -> xyz=38.472723e-3 3.257695e-3 0.000000 rpy=0 0 0.766

File: src/ah_urdf/urdf/ability_hand_right_small.urdf (robot description, URDF)
Before this commit: robot ability_hand, 47 links, 46 joints
Joints:
- joint index_q2: limit lower=0.766 upper=2.61 effort=6.0 velocity=8.0677777442 -> lower=0.00 upper=1.844 effort=6.0 velocity=8.0677777442; mimic joint=index_q1 multiplier=1.05851325 offset=0.72349796 -> joint=index_q1 multiplier=1.05851325; origin xyz=38.472723e-3 3.257695e-3 0.000000e-3 rpy=0 0 0.084474 -> xyz=38.472723e-3 3.257695e-3 0.000000e-3 rpy=0 0 0.766
- joint middle_q2: limit lower=0.766 upper=2.61 effort=6.0 velocity=8.0677777442 -> lower=0.00 upper=1.844 effort=6.0 velocity=8.0677777442; mimic joint=middle_q1 multiplier=1.05851325 offset=0.72349796 -> joint=middle_q1 multiplier=1.05851325; origin xyz=38.472723e-3 3.257695e-3 0.000000 rpy=0 0 0.084474 -> xyz=38.472723e-3 3.257695e-3 0.000000 rpy=0 0 0.766
- joint pinky_q2: limit lower=0.766 upper=2.61 effort=6.0 velocity=8.0677777442 -> lower=0.00 upper=1.844 effort=6.0 velocity=8.0677777442; mimic joint=pinky_q1 multiplier=1.05851325 offset=0.72349796 -> joint=pinky_q1 multiplier=1.05851325; origin xyz=38.472723e-3 3.257695e-3 0.000000 rpy=0 0 0.084474 -> xyz=38.472723e-3 3.257695e-3 0.000000 rpy=0 0 0.766
- joint ring_q2: limit lower=0.766 upper=2.61 effort=6.0 velocity=8.0677777442 -> lower=0.00 upper=1.844 effort=6.0 velocity=8.0677777442; mimic joint=ring_q1 multiplier=1.05851325 offset=0.72349796 -> joint=ring_q1 multiplier=1.05851325; origin xyz=38.472723e-3 3.257695e-3 0.000000 rpy=0 0 0.084474 -> xyz=38.472723e-3 3.257695e-3 0.000000 rpy=0 0 0.766

Commit message: fix urdf typo

File: src/ah_urdf/urdf/ability_hand_left_large.urdf (robot description, URDF)
Before this commit: robot ability_hand, 47 links, 46 joints
Joints:
- joint fsr29: origin xyz=0.05591 0.02160 -0.00192 -> xyz=0.05591 0.02160 -0.00192 rpy=-1.39339 0.19354 -0.40280

File: src/ah_urdf/urdf/ability_hand_left_small.urdf (robot description, URDF)
Before this commit: robot ability_hand, 47 links, 46 joints
Joints:
- joint fsr29: origin xyz=0.05591 0.02160 -0.00192 -> xyz=0.05591 0.02160 -0.00192 rpy=-1.39339 0.19354 -0.40280

File: src/ah_urdf/urdf/ability_hand_right_large.urdf (robot description, URDF)
Before this commit: robot ability_hand, 47 links, 46 joints
Joints:
- joint fsr29: origin xyz=0.05591 0.02160 0.00558 -> xyz=0.05591 0.02160 0.00558 rpy=-1.39339 0.19354 -0.40280

File: src/ah_urdf/urdf/ability_hand_right_small.urdf (robot description, URDF)
Before this commit: robot ability_hand, 47 links, 46 joints
Joints:
- joint fsr29: origin xyz=0.05591 0.02160 0.00558 -> xyz=0.05591 0.02160 0.00558 rpy=-1.39339 0.19354 -0.40280

Commit message: updated multiplier and range

File: src/ah_urdf/urdf/ability_hand_left_large.urdf (robot description, URDF)
Before this commit: robot ability_hand, 47 links, 46 joints
Joints:
- joint index_q1: limit lower=0 upper=1.74 effort=6.0 velocity=8.0677777442 -> lower=0 upper=2.00 effort=6.0 velocity=8.0677777442
- joint index_q2: mimic joint=index_q1 multiplier=1.05851325 -> joint=index_q1 multiplier=0.814
- joint middle_q1: limit lower=0 upper=1.74 effort=6.0 velocity=8.0677777442 -> lower=0 upper=2.00 effort=6.0 velocity=8.0677777442
- joint middle_q2: mimic joint=middle_q1 multiplier=1.05851325 -> joint=middle_q1 multiplier=0.814
- joint pinky_q1: limit lower=0 upper=1.74 effort=6.0 velocity=8.0677777442 -> lower=0 upper=2.00 effort=6.0 velocity=8.0677777442
- joint pinky_q2: mimic joint=pinky_q1 multiplier=1.05851325 -> joint=pinky_q1 multiplier=0.814
- joint ring_q1: limit lower=0 upper=1.74 effort=6.0 velocity=8.0677777442 -> lower=0 upper=2.00 effort=6.0 velocity=8.0677777442
- joint ring_q2: mimic joint=ring_q1 multiplier=1.05851325 -> joint=ring_q1 multiplier=0.814
- joint thumb_q1: limit lower=-1.74 upper=0 effort=1.2 velocity=40.338888721 -> lower=-2.00 upper=0 effort=1.2 velocity=40.338888721
- joint thumb_q2: limit lower=0 upper=1.74 effort=6.0 velocity=8.0677777442 -> lower=0 upper=2.00 effort=6.0 velocity=8.0677777442

File: src/ah_urdf/urdf/ability_hand_left_small.urdf (robot description, URDF)
Before this commit: robot ability_hand, 47 links, 46 joints
Joints:
- joint index_q1: limit lower=0 upper=1.74 effort=6.0 velocity=8.0677777442 -> lower=0 upper=2.00 effort=6.0 velocity=8.0677777442
- joint index_q2: mimic joint=index_q1 multiplier=1.05851325 -> joint=index_q1 multiplier=0.814
- joint middle_q1: limit lower=0 upper=1.74 effort=6.0 velocity=8.0677777442 -> lower=0 upper=2.00 effort=6.0 velocity=8.0677777442
- joint middle_q2: mimic joint=middle_q1 multiplier=1.05851325 -> joint=middle_q1 multiplier=0.814
- joint pinky_q1: limit lower=0 upper=1.74 effort=6.0 velocity=8.0677777442 -> lower=0 upper=2.00 effort=6.0 velocity=8.0677777442
- joint pinky_q2: mimic joint=pinky_q1 multiplier=1.05851325 -> joint=pinky_q1 multiplier=0.814
- joint ring_q1: limit lower=0 upper=1.74 effort=6.0 velocity=8.0677777442 -> lower=0 upper=2.00 effort=6.0 velocity=8.0677777442
- joint ring_q2: mimic joint=ring_q1 multiplier=1.05851325 -> joint=ring_q1 multiplier=0.814
- joint thumb_q1: limit lower=-1.74 upper=0 effort=1.2 velocity=40.338888721 -> lower=-2.00 upper=0 effort=1.2 velocity=40.338888721
- joint thumb_q2: limit lower=0 upper=1.74 effort=6.0 velocity=8.0677777442 -> lower=0 upper=2.00 effort=6.0 velocity=8.0677777442

File: src/ah_urdf/urdf/ability_hand_right_large.urdf (robot description, URDF)
Before this commit: robot ability_hand, 47 links, 46 joints
Joints:
- joint index_q1: limit lower=0 upper=1.74 effort=6.0 velocity=8.0677777442 -> lower=0 upper=2.00 effort=6.0 velocity=8.0677777442
- joint index_q2: mimic joint=index_q1 multiplier=1.05851325 -> joint=index_q1 multiplier=0.814
- joint middle_q1: limit lower=0 upper=1.74 effort=6.0 velocity=8.0677777442 -> lower=0 upper=2.00 effort=6.0 velocity=8.0677777442
- joint middle_q2: mimic joint=middle_q1 multiplier=1.05851325 -> joint=middle_q1 multiplier=0.814
- joint pinky_q1: limit lower=0 upper=1.74 effort=6.0 velocity=8.0677777442 -> lower=0 upper=2.00 effort=6.0 velocity=8.0677777442
- joint pinky_q2: mimic joint=pinky_q1 multiplier=1.05851325 -> joint=pinky_q1 multiplier=0.814
- joint ring_q1: limit lower=0 upper=1.74 effort=6.0 velocity=8.0677777442 -> lower=0 upper=2.00 effort=6.0 velocity=8.0677777442
- joint ring_q2: mimic joint=ring_q1 multiplier=1.05851325 -> joint=ring_q1 multiplier=0.814
- joint thumb_q1: limit lower=-1.74 upper=0 effort=1.2 velocity=40.338888721 -> lower=-2.00 upper=0 effort=1.2 velocity=40.338888721
- joint thumb_q2: limit lower=0 upper=1.74 effort=6.0 velocity=8.0677777442 -> lower=0 upper=2.00 effort=6.0 velocity=8.0677777442

File: src/ah_urdf/urdf/ability_hand_right_large_no_fsr.urdf (robot description, URDF)
Before this commit: robot ability_hand, 17 links, 16 joints
Joints:
- joint index_q1: limit lower=0 upper=1.74 effort=6.0 velocity=8.0677777442 -> lower=0 upper=2.00 effort=6.0 velocity=8.0677777442
- joint index_q2: mimic joint=index_q1 multiplier=1.05851325 -> joint=index_q1 multiplier=0.814
- joint middle_q1: limit lower=0 upper=1.74 effort=6.0 velocity=8.0677777442 -> lower=0 upper=2.00 effort=6.0 velocity=8.0677777442
- joint middle_q2: mimic joint=middle_q1 multiplier=1.05851325 -> joint=middle_q1 multiplier=0.814
- joint pinky_q1: limit lower=0 upper=1.74 effort=6.0 velocity=8.0677777442 -> lower=0 upper=2.00 effort=6.0 velocity=8.0677777442
- joint pinky_q2: mimic joint=pinky_q1 multiplier=1.05851325 -> joint=pinky_q1 multiplier=0.814
- joint ring_q1: limit lower=0 upper=1.74 effort=6.0 velocity=8.0677777442 -> lower=0 upper=2.00 effort=6.0 velocity=8.0677777442
- joint ring_q2: mimic joint=ring_q1 multiplier=1.05851325 -> joint=ring_q1 multiplier=0.814
- joint thumb_q1: limit lower=-1.74 upper=0 effort=1.2 velocity=40.338888721 -> lower=-2.00 upper=0 effort=1.2 velocity=40.338888721
- joint thumb_q2: limit lower=0 upper=1.74 effort=6.0 velocity=8.0677777442 -> lower=0 upper=2.00 effort=6.0 velocity=8.0677777442

File: src/ah_urdf/urdf/ability_hand_right_small.urdf (robot description, URDF)
Before this commit: robot ability_hand, 47 links, 46 joints
Joints:
- joint index_q1: limit lower=0 upper=1.74 effort=6.0 velocity=8.0677777442 -> lower=0 upper=2.00 effort=6.0 velocity=8.0677777442
- joint index_q2: mimic joint=index_q1 multiplier=1.05851325 -> joint=index_q1 multiplier=0.814
- joint middle_q1: limit lower=0 upper=1.74 effort=6.0 velocity=8.0677777442 -> lower=0 upper=2.00 effort=6.0 velocity=8.0677777442
- joint middle_q2: mimic joint=middle_q1 multiplier=1.05851325 -> joint=middle_q1 multiplier=0.814
- joint pinky_q1: limit lower=0 upper=1.74 effort=6.0 velocity=8.0677777442 -> lower=0 upper=2.00 effort=6.0 velocity=8.0677777442
- joint pinky_q2: mimic joint=pinky_q1 multiplier=1.05851325 -> joint=pinky_q1 multiplier=0.814
- joint ring_q1: limit lower=0 upper=1.74 effort=6.0 velocity=8.0677777442 -> lower=0 upper=2.00 effort=6.0 velocity=8.0677777442
- joint ring_q2: mimic joint=ring_q1 multiplier=1.05851325 -> joint=ring_q1 multiplier=0.814
- joint thumb_q1: limit lower=-1.74 upper=0 effort=1.2 velocity=40.338888721 -> lower=-2.00 upper=0 effort=1.2 velocity=40.338888721
- joint thumb_q2: limit lower=0 upper=1.74 effort=6.0 velocity=8.0677777442 -> lower=0 upper=2.00 effort=6.0 velocity=8.0677777442
